File: blelight-circuit/led-rfduino-rgb.kicad_pcb (KiCad board)
At the start: 2 copper layers, 44.5 x 52.1 mm, 16 parts, among them P1 POWER_REGULATOR, Q1 N_CHAN_MOSFET, Q2 N_CHAN_MOSFET, Q3 N_CHAN_MOSFET

Commit message: fixed pcb
Parts:
- removed 1PIN (x2): P***, 1pin
- added PWR1: PWR_INPUT, SIL-2, F.Cu at (138.4, 124.5)
- added USB1: USB-PROGRAMMER, SIL-6, F.Cu at (125.7, 133.3)
- moved R4 6.35 mm to (138.4, 116.8)
Connections:
- net +12V renamed N-0000012
- net GND renamed N-0000023
- BLE1 pad 14: (no net) -> N-000009
- BLE1 pad 15: (no net) -> N-0000010
- BLE1 pad 16: (no net) -> N-000007
- BLE1 pad 17: (no net) -> N-0000011
Routing:
- net N-000008: track 26.1 -> 57.2 mm
- net N-0000011: track 0.00 -> 30.1 mm, vias 0 -> 2
- net N-000007: track 0.00 -> 26.3 mm, vias 0 -> 2
- net N-0000023: track 108.6 -> 134.8 mm, vias 5 -> 8
- net N-0000013: track 28.8 -> 3.05 mm, vias 2 -> 0
- net N-0000010: track 0.00 -> 22.5 mm, vias 0 -> 2
- net N-000009: track 0.00 -> 18.7 mm, vias 0 -> 2
- net N-0000024: track 33.9 -> 50.4 mm
- net N-0000012: track 6.72 -> 17.4 mm
Other:
- board size 44.5 x 52.1 mm -> 44.5 x 55.9 mm

Commit message: lights beginnings
Other:
- net class Default: trace_width 0.254 -> 0.635
- rule pad_to_mask_clearance: 0 -> 0.0762
- rule trace_min: 0.254 -> 0.635
Changed lines of the file:
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@@
     (links 33)
     (no_connects 6)
-    (area 97.739999 81.229999 142.290001 133.400001)
+    (area 97.59982 79.936623 142.290001 137.210001)
     (thickness 1.6)
     (drawings 11)
@@
   )
   (setup
-    (last_trace_width 0.254)
+    (last_trace_width 0.635)
     (trace_clearance 0.254)
     (zone_clearance 0.508)
     (zone_45_only no)
-    (trace_min 0.254)
+    (trace_min 0.635)
     (segment_width 0.2)
     (edge_width 0.1)
@@
     (pad_size 1.778 1.778)
     (pad_drill 1.016)
-    (pad_to_mask_clearance 0)
+    (pad_to_mask_clearance 0.0762)
+    (solder_mask_min_width 0.0762)
     (aux_axis_origin 0 0)
     (visible_elements 7FFFFFFF)
     (pcbplotparams
-      (layerselection 3178497)
+      (layerselection 15761409)
       (usegerberextensions true)
       (excludeedgelayer true)
@@
       (outputformat 1)
       (mirror false)
-      (drillshape 1)
+      (drillshape 0)
       (scaleselection 1)
       (outputdirectory ""))
@@
   (net_class Default "This is the default net class."
     (clearance 0.254)
-    (trace_width 0.254)
+    (trace_width 0.635)
     (via_dia 0.889)
     (via_drill 0.635)
@@
   (gr_line (start 142.24 82.55) (end 142.24 133.35) (angle 90) (layer Edge.Cuts) (width 0.1))
   (segment (start 120.65 110.49) (end 135.89 110.49) (width 0.254) (layer F.Cu) (net 1))
-  (segment (start 114.6556 123.19) (end 119.38 123.19) (width 0.254) (layer F.Cu) (net 2) (status 400000))
-  (segment (start 127 129.54) (end 127 133.35) (width 0.254) (layer F.Cu) (net 2) (status 800000))
+  (segment (start 114.6556 123.19) (end 119.38 123.19) (width 0.254) (layer F.Cu) (net 2))
+  (segment (start 127 129.54) (end 127 133.35) (width 0.254) (layer F.Cu) (net 2))
   (via (at 127 129.54) (size 0.889) (layers F.Cu B.Cu) (net 2))
   (segment (start 119.38 129.54) (end 127 129.54) (width 0.254) (layer B.Cu) (net 2))
   (segment (start 119.38 123.19) (end 119.38 129.54) (width 0.254) (layer B.Cu) (net 2))
   (via (at 119.38 123.19) (size 0.889) (layers F.Cu B.Cu) (net 2))
-  (segment (start 132.08 133.35) (end 132.08 129.54) (width 0.254) (layer F.Cu) (net 3) (status 400000))
-  (segment (start 121.92 120.65) (end 114.6556 120.65) (width 0.254) (layer F.Cu) (net 3) (status 800000))
+  (segment (start 132.08 133.35) (end 132.08 129.54) (width 0.254) (layer F.Cu) (net 3))
+  (segment (start 121.92 120.65) (end 114.6556 120.65) (width 0.254) (layer F.Cu) (net 3))
   (via (at 121.92 120.65) (size 0.889) (layers F.Cu B.Cu) (net 3))
   (segment (start 121.92 124.46) (end 121.92 120.65) (width 0.254) (layer B.Cu) (net 3))
@@
   (segment (start 125.73 121.031) (end 125.73 124.079) (width 0.254) (layer F.Cu) (net 5))
   (segment (start 120.65 87.63) (end 135.89 87.63) (width 0.254) (layer F.Cu) (net 6))
-  (segment (start 114.6556 127) (end 110.49 127) (width 0.254) (layer F.Cu) (net 7) (status 400000))
-  (segment (start 110.49 133.35) (end 119.38 133.35) (width 0.254) (layer F.Cu) (net 7) (status 800000))
+  (segment (start 114.6556 127) (end 110.49 127) (width 0.254) (layer F.Cu) (net 7))
+  (segment (start 110.49 133.35) (end 119.38 133.35) (width 0.254) (layer F.Cu) (net 7))
   (via (at 110.49 133.35) (size 0.889) (layers F.Cu B.Cu) (net 7))
   (segment (start 110.49 127) (end 110.49 133.35) (width 0.254) (layer B.Cu) (net 7))
   (via (at 110.49 127) (size 0.889) (layers F.Cu B.Cu) (net 7))
-  (segment (start 131.191 113.03) (end 131.191 115.189) (width 0.254) (layer F.Cu) (net 7) (status 400000))
+  (segment (start 131.191 113.03) (end 131.191 115.189) (width 0.254) (layer F.Cu) (net 7))
   (segment (start 131.191 115.189) (end 128.27 118.11) (width 0.254) (layer F.Cu) (net 7))
-  (segment (start 128.27 123.19) (end 132.08 123.19) (width 0.254) (layer F.Cu) (net 7) (status 800000))
+  (segment (start 128.27 123.19) (end 132.08 123.19) (width 0.254) (layer F.Cu) (net 7))
   (via (at 128.27 123.19) (size 0.889) (layers F.Cu B.Cu) (net 7))
   (segment (start 128.27 118.11) (end 128.27 123.19) (width 0.254) (layer B.Cu) (net 7))
@@
   (segment (start 118.11 100.33) (end 113.03 105.41) (width 0.254) (layer F.Cu) (net 12))
   (segment (start 118.11 90.17) (end 118.11 100.33) (width 0.254) (layer F.Cu) (net 12))
-  (segment (start 114.6556 121.92) (end 120.65 121.92) (width 0.254) (layer F.Cu) (net 13) (status 400000))
-  (segment (start 129.54 130.81) (end 129.54 133.35) (width 0.254) (layer F.Cu) (net 13) (status 800000))
+  (segment (start 114.6556 121.92) (end 120.65 121.92) (width 0.254) (layer F.Cu) (net 13))
+  (segment (start 129.54 130.81) (end 129.54 133.35) (width 0.254) (layer F.Cu) (net 13))
   (via (at 129.54 130.81) (size 0.889) (layers F.Cu B.Cu) (net 13))
   (segment (start 128.27 130.81) (end 129.54 130.81) (width 0.254) (layer B.Cu) (net 13))
@@
   (segment (start 120.65 121.92) (end 120.65 128.27) (width 0.254) (layer B.Cu) (net 13))
   (via (at 120.65 121.92) (size 0.889) (layers F.Cu B.Cu) (net 13))
-  (segment (start 114.6556 125.73) (end 109.22 125.73) (width 0.254) (layer F.Cu) (net 14) (status 400000))
-  (segment (start 121.92 135.89) (end 121.92 133.35) (width 0.254) (layer F.Cu) (net 14) (status 800000))
+  (segment (start 114.6556 125.73) (end 109.22 125.73) (width 0.254) (layer F.Cu) (net 14))
+  (segment (start 121.92 135.89) (end 121.92 133.35) (width 0.254) (layer F.Cu) (net 14))
   (via (at 121.92 135.89) (size 0.889) (layers F.Cu B.Cu) (net 14))
   (segment (start 109.22 135.89) (end 121.92 135.89) (width 0.254) (layer B.Cu) (net 14))
   (segment (start 109.22 125.73) (end 109.22 135.89) (width 0.254) (layer B.Cu) (net 14))
   (via (at 109.22 125.73) (size 0.889) (layers F.Cu B.Cu) (net 14))
-  (segment (start 114.6556 125.73) (end 123.19 125.73) (width 0.254) (layer F.Cu) (net 14) (status 400000))
-  (segment (start 123.571 117.729) (end 125.73 117.729) (width 0.254) (layer F.Cu) (net 14) (status 800000))
+  (segment (start 114.6556 125.73) (end 123.19 125.73) (width 0.254) (layer F.Cu) (net 14))
+  (segment (start 123.571 117.729) (end 125.73 117.729) (width 0.254) (layer F.Cu) (net 14))
   (segment (start 123.19 118.11) (end 123.571 117.729) (width 0.254) (layer F.Cu) (net 14))
   (segment (start 123.19 125.73) (end 123.19 118.11) (width 0.254) (layer F.Cu) (net 14))
   (segment (start 132.08 120.65) (end 128.651 120.65) (width 0.254) (layer F.Cu) (net 14))
   (segment (start 128.651 120.65) (end 125.73 117.729) (width 0.254) (layer F.Cu) (net 14))
-  (segment (start 114.6556 124.46) (end 118.11 124.46) (width 0.254) (layer F.Cu) (net 15) (status 400000))
-  (segment (start 124.46 130.81) (end 124.46 133.35) (width 0.254) (layer F.Cu) (net 15) (status 800000))
+  (segment (start 114.6556 124.46) (end 118.11 124.46) (width 0.254) (layer F.Cu) (net 15))
+  (segment (start 124.46 130.81) (end 124.46 133.35) (width 0.254) (layer F.Cu) (net 15))
   (via (at 124.46 130.81) (size 0.889) (layers F.Cu B.Cu) (net 15))
   (segment (start 118.11 130.81) (end 124.46 130.81) (width 0.254) (layer B.Cu) (net 15))

Commit message: lightserver working
Parts:
- added R6: 39, 3W, SM1206, F.Cu at (129.5, 99.1)
- added R7: 39, 3W, SM1206, F.Cu at (129.5, 110.5)
- R1, R2, R3: value 10k -> 20k
- R4: value 3ohm 1W -> 13.9, 2W
- moved R4 30.5 mm to (129.5, 87.6), turned to 180 degrees
Connections:
- BLE1 pad 5: N-000004 (its old number) -> N-000005
- D1 pad 2: N-000002 (its old number) -> N-0000012
- D2 pad 2: N-000003 (its old number) -> N-000005
- D3 pad 2: N-000001 (its old number) -> N-000009
- P1 pad 1: N-0000012 -> N-0000024
- PWR1 pad 1: N-0000012 -> N-0000024
- Q1 pad 3: N-000002 (its old number) -> N-0000013
- Q2 pad 3: N-000003 (its old number) -> N-0000011
- Q3 pad 2: N-000004 (its old number) -> N-000005
- Q3 pad 3: N-000001 (its old number) -> N-0000010
- R3 pad 1: N-000004 (its old number) -> N-000005
- R4 pad 1: N-0000024 -> N-0000012
- R4 pad 2: N-0000012 -> N-0000013
Routing:
- net N-000005: track 0.00 -> 35.6 mm, vias 0 -> 2
- net N-000004 (its old number): track 29.6 -> 0.00 mm
- net N-000003 (its old number): track 15.2 -> 0.00 mm
- net N-000002 (its old number): track 15.2 -> 0.00 mm
- net N-000001 (its old number): track 15.2 -> 0.00 mm
- net N-0000012: track 17.4 -> 4.70 mm
- net N-0000013: track 0.00 -> 7.24 mm
- net N-0000011: track 0.00 -> 7.24 mm
- net N-0000010: track 0.00 -> 7.24 mm
- net N-000009: track 0.00 -> 4.70 mm
- net N-0000024: track 50.4 -> 48.0 mm
- net N-000003: track 48.4 -> 46.2 mm, vias 0 -> 2
- net N-000007: track 134.8 -> 133.0 mm, vias 8 -> 7
- net N-000004: track 38.3 -> 38.8 mm, vias 0 -> 2

Commit message: removed corners
Parts:
- removed R5: 30k, SM1206
- removed VR1: 10Mohm, SM1206
Connections:
- BLE1 pad 5: N-000005 (its old number) -> N-000003
- BLE1 pad 6: N-0000023 -> (no net)
- D2 pad 2: N-000005 (its old number) -> N-000009
- Q3 pad 2: N-000005 (its old number) -> N-000003
- R3 pad 1: N-000005 (its old number) -> N-000003
- R6 pad 1: N-000005 (its old number) -> N-000009
Routing:
- net N-000005 (its old number): track 35.6 -> 0.00 mm, vias 2 -> 0
- net N-000003: track 0.00 -> 30.9 mm, vias 0 -> 2
- net N-0000011: track 30.1 -> 24.9 mm
- net N-000009: track 0.00 -> 4.70 mm
- net N-0000012: track 26.3 -> 21.9 mm
- net N-0000025: track 133.0 -> 137.1 mm
- net N-000001: track 18.7 -> 15.0 mm
- net N-0000013: track 22.5 -> 18.8 mm
- net N-0000023: track 3.05 -> 0.00 mm
- net N-0000016: track 57.2 -> 59.0 mm
- net N-000006: track 46.2 -> 47.5 mm
